File: pcb/GestureControl/GestureControl.sch (KiCad schematic (older format))
At the start: 2 parts

Commit message: add
Parts:
- removed U?: STM32F401RETx, Package_QFP:LQFP-64_10x10mm_P0.5mm, symbol MCU_ST_STM32F4:STM32F401RETx
- added 10k: R, symbol Device:R
- added C? (x4): CP, symbol Device:CP
- added D? (x5): LED, symbol Device:LED
- added D?: D, symbol Device:D
- added J? (x2): Conn_01x08, symbol Connector_Generic:Conn_01x08
- added J?: Conn_01x06, symbol Connector_Generic:Conn_01x06
- added J?: Conn_01x10, symbol Connector_Generic:Conn_01x10
- added R? (x5): 100, symbol Device:R
- added R?: 10k, symbol Device:R
- added SW? (x2): SW_Push, symbol Switch:SW_Push
- added U?: VL53L3CXV0DH_1, QFN_CXV0DH/1_STM, symbol VL53L3CX:VL53L3CXV0DH_1
- added U?: AMS1117-5.0, Package_TO_SOT_SMD:SOT-223-3_TabPin2, symbol Regulator_Linear:AMS1117-5.0
Connections:
- net labels added: +3.3V, +5V, GND, GPIOI_0, GPIOI_1, GPIOI_2, LED_1, LED_2, LED_3, LED_4, LED_5, SCL, SDA, SW_1, SW_2, VCC, XSHUT_0, XSHUT_1, XSHUT_2
- wire segments 0 -> 69
Other:
- note added: "peripherals"
- moved on the sheet: U?

Commit message: end simple schematic
Parts:
- added C? (x6): 100n, symbol Device:C
- added C? (x3): 4.7µ, symbol Device:C
- added C?: 10µ, symbol Device:CP
- added D?: 1N4002, symbol Device:D
- added J?: Screw_Terminal_01x02, symbol Connector:Screw_Terminal_01x02
- added J?: Conn_01x02, symbol Connector_Generic:Conn_01x02
- added R? (x2): 4k7, symbol Device:R
- added R? (x6): 10k, symbol Device:R
- added U?: VL53L3CXV0DH_CENTER, QFN_CXV0DH/1_STM, symbol VL53L3CX:VL53L3CXV0DH_1
- added U?: VL53L3CXV0DH_RIGHT, QFN_CXV0DH/1_STM, symbol VL53L3CX:VL53L3CXV0DH_1
- C? (x2): value CP -> 100µ
- C? (x2): value CP -> 10µ
- D?: value D -> 1N4002
- R?: renamed from 10k; value R -> 10k
- SW?: value SW_Push -> SW_1
- SW?: value SW_Push -> SW_2
- U?: value VL53L3CXV0DH_1 -> VL53L3CXV0DH_LEFT
Connections:
- wire segments 69 -> 158
Other:
- note added: "connectors"
- note added: "data"
- note added: "power"
- moved on the sheet: J?, U?

Commit message: add MCU + PCB
Parts:
- removed C? (x6): 100n, symbol Device:C
- removed C? (x3): 4.7µ, symbol Device:C
- removed J?: Conn_01x02, symbol Connector_Generic:Conn_01x02
- removed R? (x7): 10k, symbol Device:R
- removed SW?: SW_1, symbol Switch:SW_Push
- removed SW?: SW_2, symbol Switch:SW_Push
- removed U?: VL53L3CXV0DH_LEFT, QFN_CXV0DH/1_STM, symbol VL53L3CX:VL53L3CXV0DH_1
- removed U?: VL53L3CXV0DH_CENTER, QFN_CXV0DH/1_STM, symbol VL53L3CX:VL53L3CXV0DH_1
- removed U?: VL53L3CXV0DH_RIGHT, QFN_CXV0DH/1_STM, symbol VL53L3CX:VL53L3CXV0DH_1
- added C23, C24: 100n, Capacitor_SMD:C_0805_2012Metric_Pad1.18x1.45mm_HandSolder, symbol Device:C
- added J2: Conn_01x04_I2I-LCD, Connector_PinHeader_2.54mm:PinHeader_1x04_P2.54mm_Vertical, symbol Connector_Generic:Conn_01x04
- added R19, R20: 100, Resistor_SMD:R_0805_2012Metric_Pad1.20x1.40mm_HandSolder, symbol Device:R
- added R7: 10k, Resistor_SMD:R_0805_2012Metric_Pad1.20x1.40mm_HandSolder, symbol Device:R
- added SW1, SW2: SW_Push_Dual, symbol Switch:SW_Push_Dual
- D1, D2, D3, D4, D5: renamed from D?; footprint (none) -> LED_SMD:LED_0805_2012Metric_Pad1.15x1.40mm_HandSolder
- J3, J6: renamed from J?; footprint (none) -> Connector_PinHeader_2.54mm:PinHeader_1x08_P2.54mm_Vertical
- J4: renamed from J?; footprint (none) -> Connector_PinHeader_2.54mm:PinHeader_1x06_P2.54mm_Vertical
- J5: renamed from J?; footprint (none) -> Connector_PinHeader_2.54mm:PinHeader_1x10_P2.54mm_Vertical
- R1, R2, R3, R4, R5, R6, R8, R9: renamed from R?; footprint (none) -> Resistor_SMD:R_0805_2012Metric_Pad1.20x1.40mm_HandSolder
- gave numbers to parts that had none: 10
Connections:
- wire segments 158 -> 119
Other:
- note added: "mcu"
- note added: "sensors"
- moved on the sheet: C1, C2, C3, C4, C5, D6, D7, J1, J3, J4, R6, R8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

Commit message: add
Parts:
- C1, C2, C3, C4, C5: footprint (none) -> Capacitor_SMD:CP_Elec_6.3x5.4
- C23, C24: footprint Capacitor_SMD:C_0805_2012Metric_Pad1.18x1.45mm_HandSolder -> Capacitor_SMD:C_0603_1608Metric_Pad1.08x0.95mm_HandSolder
- D1: value LED -> L1
- D2: value LED -> L2
- D3: value LED -> L3
- D4: value LED -> L4
- D5: value LED -> L5
- D6, D7: footprint (none) -> Diode_SMD:D_SMA_Handsoldering
- J1: value Screw_Terminal_01x02 -> BATT; footprint (none) -> Connector_Phoenix_MC:PhoenixContact_MC_1,5_2-G-3.5_1x02_P3.50mm_Horizontal
- J2: footprint Connector_PinHeader_2.54mm:PinHeader_1x04_P2.54mm_Vertical -> Connector_PinSocket_2.54mm:PinSocket_1x04_P2.54mm_Vertical
- SW1: value SW_Push_Dual -> SW1; footprint (none) -> Button_Switch_SMD:SW_Push_1P1T_NO_6x6mm_H9.5mm
- SW2: value SW_Push_Dual -> SW2; footprint (none) -> Button_Switch_SMD:SW_Push_1P1T_NO_6x6mm_H9.5mm
- U1: value AMS1117-3.3 -> LD1117-3.3
- U2: value AMS1117-5.0 -> LD1117-5.0
Connections:
- net +5V: now also C1.1, U1.3 (VI)
- net VCC: no longer C1.1, U1.3 (VI)
Changed lines of the file:
@@
 P 5900 1100
 F 0 "U1" H 5900 1342 50  0000 C CNN
-F 1 "AMS1117-3.3" H 5900 1251 50  0000 C CNN
+F 1 "LD1117-3.3" H 5900 1251 50  0000 C CNN
 F 2 "Package_TO_SOT_SMD:SOT-223-3_TabPin2" H 5900 1300 50  0001 C CNN
 F 3 "http://www.advanced-monolithic.com/pdf/ds1117.pdf" H 6000 850 50  0001 C CNN
@@
 P 5900 2150
 F 0 "U2" H 5900 2392 50  0000 C CNN
-F 1 "AMS1117-5.0" H 5900 2301 50  0000 C CNN
+F 1 "LD1117-5.0" H 5900 2301 50  0000 C CNN
 F 2 "Package_TO_SOT_SMD:SOT-223-3_TabPin2" H 5900 2350 50  0001 C CNN
 F 3 "http://www.advanced-monolithic.com/pdf/ds1117.pdf" H 6000 1900 50  0001 C CNN
@@
 P 1750 1250
 F 0 "D1" H 1743 995 50  0000 C CNN
-F 1 "LED" H 1743 1086 50  0000 C CNN
+F 1 "L1" H 1743 1086 50  0000 C CNN
 F 2 "LED_SMD:LED_0805_2012Metric_Pad1.15x1.40mm_HandSolder" H 1750 1250 50  0001 C CNN
 F 3 "~" H 1750 1250 50  0001 C CNN
@@
 P 1750 1700
 F 0 "D2" H 1743 1445 50  0000 C CNN
-F 1 "LED" H 1743 1536 50  0000 C CNN
+F 1 "L2" H 1743 1536 50  0000 C CNN
 F 2 "LED_SMD:LED_0805_2012Metric_Pad1.15x1.40mm_HandSolder" H 1750 1700 50  0001 C CNN
 F 3 "~" H 1750 1700 50  0001 C CNN
@@
 P 1750 2150
 F 0 "D3" H 1743 1895 50  0000 C CNN
-F 1 "LED" H 1743 1986 50  0000 C CNN
+F 1 "L3" H 1743 1986 50  0000 C CNN
 F 2 "LED_SMD:LED_0805_2012Metric_Pad1.15x1.40mm_HandSolder" H 1750 2150 50  0001 C CNN
 F 3 "~" H 1750 2150 50  0001 C CNN
@@
 P 1750 2600
 F 0 "D4" H 1743 2345 50  0000 C CNN
-F 1 "LED" H 1743 2436 50  0000 C CNN
+F 1 "L4" H 1743 2436 50  0000 C CNN
 F 2 "LED_SMD:LED_0805_2012Metric_Pad1.15x1.40mm_HandSolder" H 1750 2600 50  0001 C CNN
 F 3 "~" H 1750 2600 50  0001 C CNN
@@
 P 1750 3050
 F 0 "D5" H 1743 2795 50  0000 C CNN
-F 1 "LED" H 1743 2886 50  0000 C CNN
+F 1 "L5" H 1743 2886 50  0000 C CNN
 F 2 "LED_SMD:LED_0805_2012Metric_Pad1.15x1.40mm_HandSolder" H 1750 3050 50  0001 C CNN
 F 3 "~" H 1750 3050 50  0001 C CNN
@@
 Wire Wire Line
 	5900 1500 5900 1400
-$Comp
-L Device:CP C3
-U 1 1 62130130
-P 6400 1300
-F 0 "C3" H 6518 1346 50  0000 L CNN
-F 1 "100µ" H 6518 1255 50  0000 L CNN
-F 2 "" H 6438 1150 50  0001 C CNN
-F 3 "~" H 6400 1300 50  0001 C CNN
-	1    6400 1300
-	1    0    0    -1
-$EndComp
-$Comp
-L Device:CP C1
-U 1 1 621309F0
-P 5400 1300
-F 0 "C1" H 5518 1346 50  0000 L CNN
-F 1 "10µ" H 5518 1255 50  0000 L CNN
-F 2 "" H 5438 1150 50  0001 C CNN
-F 3 "~" H 5400 1300 50  0001 C CNN
-	1    5400 1300
-	1    0    0    -1
-$EndComp
 Wire Wire Line
 	5400 1150 5400 1100
@@
 Wire Wire Line
 	6400 1100 6400 1150
-$Comp
-L Device:CP C4
-U 1 1 621320C1
-P 6400 2350
-F 0 "C4" H 6518 2396 50  0000 L CNN
-F 1 "100µ" H 6518 2305 50  0000 L CNN
-F 2 "" H 6438 2200 50  0001 C CNN
-F 3 "~" H 6400 2350 50  0001 C CNN
-	1    6400 2350
-	1    0    0    -1
-$EndComp
-$Comp
-L Device:CP C2
-U 1 1 6213274A
-P 5400 2350
-F 0 "C2" H 5518 2396 50  0000 L CNN
-F 1 "10µ" H 5518 2305 50  0000 L CNN
-F 2 "" H 5438 2200 50  0001 C CNN
-F 3 "~" H 5400 2350 50  0001 C CNN
-	1    5400 2350
-	1    0    0    -1
-$EndComp
 Wire Wire Line
 	5400 2200 5400 2150
@@
 F 0 "D7" H 6600 1933 50  0000 C CNN
 F 1 "1N4002" H 6600 2024 50  0000 C CNN
-F 2 "" H 6600 2150 50  0001 C CNN
+F 2 "Diode_SMD:D_SMA_Handsoldering" H 6600 2150 50  0001 C CNN
 F 3 "~" H 6600 2150 50  0001 C CNN
 	1    6600 2150
@@
 F 3 "" H 5200 2100 50  0001 C CNN
 	1    5200 2100
-	1    0    0    -1
-$EndComp
-$Comp
-L power:VCC #PWR0109
-U 1 1 6214288C
-P 5200 1050
-F 0 "#PWR0109" H 5200 900 50  0001 C CNN
-F 1 "VCC" H 5215 1223 50  0000 C CNN
-F 2 "" H 5200 1050 50  0001 C CNN
-F 3 "" H 5200 1050 50  0001 C CNN
-	1    5200 1050
 	1    0    0    -1
 $EndComp
@@
 P 5500 3350
 F 0 "J1" H 5650 3200 50  0000 C CNN
-F 1 "Screw_Terminal_01x02" H 5450 3050 50  0000 C CNN
-F 2 "" H 5500 3350 50  0001 C CNN
+F 1 "BATT" H 5450 3050 50  0000 C CNN
+F 2 "Connector_Phoenix_MC:PhoenixContact_MC_1,5_2-G-3.5_1x02_P3.50mm_Horizontal" H 5500 3350 50  0001 C CNN
 F 3 "~" H 5500 3350 50  0001 C CNN
 	1    5500 3350
@@
 F 0 "C5" H 6718 3346 50  0000 L CNN
 F 1 "10µ" H 6718 3255 50  0000 L CNN
-F 2 "" H 6638 3150 50  0001 C CNN
+F 2 "Capacitor_SMD:CP_Elec_6.3x5.4" H 6638 3150 50  0001 C CNN
 F 3 "~" H 6600 3300 50  0001 C CNN
 	1    6600 3300
@@
 F 0 "D6" H 6000 2883 50  0000 C CNN
 F 1 "1N4002" H 6000 2974 50  0000 C CNN
-F 2 "" H 6000 3100 50  0001 C CNN
+F 2 "Diode_SMD:D_SMA_Handsoldering" H 6000 3100 50  0001 C CNN
 F 3 "~" H 6000 3100 50  0001 C CNN
 	1    6000 3100
@@
 P 2950 1400
 F 0 "SW1" H 2950 1685 50  0000 C CNN
-F 1 "SW_Push_Dual" H 2950 1594 50  0000 C CNN
-F 2 "" H 2950 1600 50  0001 C CNN
+F 1 "SW1" H 2950 1594 50  0000 C CNN
+F 2 "Button_Switch_SMD:SW_Push_1P1T_NO_6x6mm_H9.5mm" H 2950 1600 50  0001 C CNN
 F 3 "~" H 2950 1600 50  0001 C CNN
 	1    2950 1400
@@
 F 0 "J2" H 1630 3792 50  0000 L CNN
 F 1 "Conn_01x04_I2I-LCD" H 1200 4050 50  0000 L CNN
-F 2 "Connector_PinHeader_2.54mm:PinHeader_1x04_P2.54mm_Vertical" H 1550 3800 50  0001 C CNN
+F 2 "Connector_PinSocket_2.54mm:PinSocket_1x04_P2.54mm_Vertical" H 1550 3800 50  0001 C CNN
 F 3 "~" H 1550 3800 50  0001 C CNN
 	1    1550 3800
@@
 F 0 "C23" V 2698 1950 50  0000 C CNN
 F 1 "100n" V 2789 1950 50  0000 C CNN
-F 2 "Capacitor_SMD:C_0805_2012Metric_Pad1.18x1.45mm_HandSolder" H 2988 1800 50  0001 C CNN
+F 2 "Capacitor_SMD:C_0603_1608Metric_Pad1.08x0.95mm_HandSolder" H 2988 1800 50  0001 C CNN
 F 3 "~" H 2950 1950 50  0001 C CNN
 	1    2950 1950
@@
 P 2950 2550
 F 0 "SW2" H 2950 2835 50  0000 C CNN
-F 1 "SW_Push_Dual" H 2950 2744 50  0000 C CNN
-F 2 "" H 2950 2750 50  0001 C CNN
+F 1 "SW2" H 2950 2744 50  0000 C CNN
+F 2 "Button_Switch_SMD:SW_Push_1P1T_NO_6x6mm_H9.5mm" H 2950 2750 50  0001 C CNN
 F 3 "~" H 2950 2750 50  0001 C CNN
 	1    2950 2550
@@
 F 0 "C24" V 2698 3100 50  0000 C CNN
 F 1 "100n" V 2789 3100 50  0000 C CNN
-F 2 "Capacitor_SMD:C_0805_2012Metric_Pad1.18x1.45mm_HandSolder" H 2988 2950 50  0001 C CNN
+F 2 "Capacitor_SMD:C_0603_1608Metric_Pad1.08x0.95mm_HandSolder" H 2988 2950 50  0001 C CNN
 F 3 "~" H 2950 3100 50  0001 C CNN
 	1    2950 3100
@@
 Wire Notes Line
 	700  4200 3650 4200
+$Comp
+L Device:CP C2
+U 1 1 6213274A
+P 5400 2350
+F 0 "C2" H 5518 2396 50  0000 L CNN
+F 1 "10µ" H 5518 2305 50  0000 L CNN
+F 2 "Capacitor_SMD:CP_Elec_6.3x5.4" H 5438 2200 50  0001 C CNN
+F 3 "~" H 5400 2350 50  0001 C CNN
+	1    5400 2350
+	1    0    0    -1
+$EndComp
+$Comp
+L Device:CP C4
+U 1 1 621320C1
+P 6400 2350
+F 0 "C4" H 6518 2396 50  0000 L CNN
+F 1 "100µ" H 6518 2305 50  0000 L CNN
+F 2 "Capacitor_SMD:CP_Elec_6.3x5.4" H 6438 2200 50  0001 C CNN
+F 3 "~" H 6400 2350 50  0001 C CNN
+	1    6400 2350
+	1    0    0    -1
+$EndComp
+$Comp
+L Device:CP C3
+U 1 1 62130130
+P 6400 1300
+F 0 "C3" H 6518 1346 50  0000 L CNN
+F 1 "100µ" H 6518 1255 50  0000 L CNN
+F 2 "Capacitor_SMD:CP_Elec_6.3x5.4" H 6438 1150 50  0001 C CNN
+F 3 "~" H 6400 1300 50  0001 C CNN
+	1    6400 1300
+	1    0    0    -1
+$EndComp
+$Comp
+L Device:CP C1
+U 1 1 621309F0
+P 5400 1300
+F 0 "C1" H 5518 1346 50  0000 L CNN
+F 1 "10µ" H 5518 1255 50  0000 L CNN
+F 2 "Capacitor_SMD:CP_Elec_6.3x5.4" H 5438 1150 50  0001 C CNN
+F 3 "~" H 5400 1300 50  0001 C CNN
+	1    5400 1300
+	1    0    0    -1
+$EndComp
+$Comp
+L power:+5V #PWR0109
+U 1 1 62285A43
+P 5200 1050
+F 0 "#PWR0109" H 5200 900 50  0001 C CNN
+F 1 "+5V" H 5215 1223 50  0000 C CNN
+F 2 "" H 5200 1050 50  0001 C CNN
+F 3 "" H 5200 1050 50  0001 C CNN
+	1    5200 1050
+	1    0    0    -1
+$EndComp
 $EndSCHEMATC

Commit message: new PCB
Parts:
- added H1, H2, H3, H4, H5, H6: MountingHole, MountingHole:MountingHole_3.2mm_M3, symbol Mechanical:MountingHole
- added R21, R22: 4k7, Resistor_SMD:R_0805_2012Metric_Pad1.20x1.40mm_HandSolder, symbol Device:R
- J1: renamed from J2; footprint Connector_PinSocket_2.54mm:PinSocket_1x04_P2.54mm_Vertical -> Connector_PinHeader_2.54mm:PinHeader_1x04_P2.54mm_Vertical
- renumbered C23 to C1, C24 to C2, C1 to C3, C2 to C4, C3 to C5, C4 to C6, C5 to C7, J1 to J2, R8 to R10, R9 to R11, R19 to R8, R20 to R9
Connections:
- net +3V3: now also R21.1, R22.1
- net SCL renamed SCL1
- net SDA renamed SDA1
- new net SCL2: R22.2
- new net SDA2: R21.2
