File: pcb/GestureControl/GestureControl.sch (KiCad schematic (older format))
At the start: 43 parts, among them J1 Conn_01x04_I2I-LCD, J2 BATT, J3 Conn_01x08, J4 Conn_01x06, J5 Conn_01x10, J6 Conn_01x08, SW1 SW1, SW2 SW2, U1 LD1117-3.3, U2 LD1117-5.0

Commit message: add feedback Philip
Parts:
- added C34: 4.7µ, Capacitor_SMD:C_0805_2012Metric_Pad1.18x1.45mm_HandSolder, symbol Device:C
Connections:
- net +3V3: now also C34.1
- net GND: now also C34.2
Other:
- moved on the sheet: C3, C4, C5, C6, C7, D6, D7, J2, U1, U2

Commit message: werking printf()
Other:
- note added: "Arduino Header connectors"
- note removed: "connectors"
- moved on the sheet: C3, C34, C4, C5, C6, C7, D6, D7, J2, J3, J4, J5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

Commit message: add PCBV0.11
Parts:
- removed C3, C4: 10µ, Capacitor_SMD:CP_Elec_6.3x5.4, symbol Device:CP
- removed C5, C6: 100µ, Capacitor_SMD:CP_Elec_6.3x5.4, symbol Device:CP
- removed D7: 1N4002, Diode_SMD:D_SMA_Handsoldering, symbol Device:D
- removed U1: LD1117-3.3, Package_TO_SOT_SMD:SOT-223-3_TabPin2, symbol Regulator_Linear:AMS1117-3.3
- removed U2: LD1117-5.0, Package_TO_SOT_SMD:SOT-223-3_TabPin2, symbol Regulator_Linear:AMS1117-5.0
- added C13: 10µ, Capacitor_SMD:C_1206_3216Metric_Pad1.33x1.80mm_HandSolder, symbol Device:C
- added C3, C4: 10µF, Capacitor_SMD:C_1206_3216Metric_Pad1.33x1.80mm_HandSolder, symbol Device:C
- added C5, C6: 100nF, Capacitor_SMD:C_0603_1608Metric_Pad1.08x0.95mm_HandSolder, symbol Device:C
- added D7, D8: B230A, Diode_SMD:D_SMA_Handsoldering, symbol Device:D_Schottky
- added JP1, JP10, JP11, JP12, JP14, JP4, JP5, JP6, JP7, JP8, JP9: SolderJumper_2_Open, Jumper:SolderJumper-2_P1.3mm_Open_Pad1.0x1.5mm, symbol Jumper:SolderJumper_2_Open
- added L1, L2: 10µH, Inductor_SMD:L_Taiyo-Yuden_NR-50xx_HandSoldering, symbol Device:L
- added R14, R15: 100k, Resistor_SMD:R_0805_2012Metric_Pad1.20x1.40mm_HandSolder, symbol Device:R
- added R18: 220, Resistor_SMD:R_0805_2012Metric_Pad1.20x1.40mm_HandSolder, symbol Device:R
- added R19: 820, Resistor_SMD:R_0805_2012Metric_Pad1.20x1.40mm_HandSolder, symbol Device:R
- added R23, R24: 100, Resistor_SMD:R_0805_2012Metric_Pad1.20x1.40mm_HandSolder, symbol Device:R
- added R25: 18k, Resistor_SMD:R_0805_2012Metric_Pad1.20x1.40mm_HandSolder, symbol Device:R
- added R26: 10k, Resistor_SMD:R_0805_2012Metric_Pad1.20x1.40mm_HandSolder, symbol Device:R
- added R27, R28: 56k, Resistor_SMD:R_0805_2012Metric_Pad1.20x1.40mm_HandSolder, symbol Device:R
- added U1, U2: AP5100_3.3, Package_TO_SOT_SMD:TSOT-23-6_HandSoldering, symbol AP5100:AP5100
- C34: value 4.7µ -> 10µ; footprint Capacitor_SMD:C_0805_2012Metric_Pad1.18x1.45mm_HandSolder -> Capacitor_SMD:C_1206_3216Metric_Pad1.33x1.80mm_HandSolder
Connections:
- net +3V3: now also C13.1, L1.2, R27.2; no longer C34.1
- net +5V: now also C34.1, L2.2, R28.2
- net GND: now also C13.2, C3.2, C4.2, D7.2 (A), D8.2 (A), R18.2, R19.2, U1.2 (GND), U2.2 (GND)
- net VCC: now also C3.1, C4.1, R14.1, R15.1, U1.5 (IN), U2.5 (IN)
- net XSHUT_0: now also JP5.2 (B); no longer J5.1 (Pin_1)
- net XSHUT_1: now also JP11.1 (A); no longer J6.8 (Pin_8)
- net XSHUT_2: now also JP8.1 (A); no longer J6.5 (Pin_5)
- net _XSHUT_0: now reaches J4.4 (Pin_4)
- net _XSHUT_0: now also JP5.1 (A)
- net _XSHUT_3: now reaches J4.5 (Pin_5)
- net _XSHUT_3: now also JP6.1 (A)
- net _XSHUT_6: now reaches J4.6 (Pin_6)
- net _XSHUT_6: now also JP7.1 (A)
- net _XSHUT_8: now reaches J5.3 (Pin_3)
- net _XSHUT_8: now also JP10.2 (B)
- net _XSHUT_5: now reaches J5.4 (Pin_4)
- net _XSHUT_5: now also JP9.2 (B)
- net _XSHUT_2: now reaches J5.5 (Pin_5)
- net _XSHUT_2: now also JP8.2 (B)
- new net: C5.2, U1.1 (BST)
- new net: R25.1, R27.1, U1.3 (FB)
- new net: JP1.1 (A), R14.2
- new net: C5.1, R23.2
- new net: R18.1, R25.2
- new net: C6.2, U2.1 (BST)
- new net: R26.1, R28.1, U2.3 (FB)
- new net: JP4.1 (A), R15.2
- new net: C6.1, R24.2
- new net: R19.1, R26.2
- new net BUCK_33_EN: JP1.2 (B), U1.4 (EN)
- new net BUCK_5_EN: JP4.2 (B), U2.4 (EN)
- new net OUT3.3: D7.1 (K), L1.1, R23.1, U1.6 (OUT)
- new net OUT5.0: D8.1 (K), L2.1, R24.1, U2.6 (OUT)
- new net XSHUT_3: JP6.2 (B)
- new net XSHUT_4: JP12.1 (A)
- new net XSHUT_5: JP9.1 (A)
- new net XSHUT_6: JP7.2 (B)
- new net XSHUT_7: JP14.1 (A)
- new net XSHUT_8: JP10.1 (A)
- new net _XSHUT_1: J5.1 (Pin_1), JP11.2 (B)
- new net _XSHUT_4: J6.8 (Pin_8), JP12.2 (B)
- new net _XSHUT_7: J6.5 (Pin_5), JP14.2 (B)
Other:
- moved on the sheet: C1, C2, C7, D1, D2, D3, D4, D5, D6, H1, H2, H3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

Commit message: update board design
Parts:
- added C11, C12: 4.7µF, Capacitor_SMD:C_0805_2012Metric_Pad1.18x1.45mm_HandSolder, symbol Device:C
Connections:
- net +3V3: now also C11.1, C12.1
- net GND: now also C11.2, C12.2
Other:
- moved on the sheet: R10, R11, R21, R22
Changed lines of the file:
@@
 Wire Wire Line
 	8500 5500 8450 5500
-Text GLabel 7750 1250 0    50   Input ~ 0
+Text GLabel 8550 1250 0    50   Input ~ 0
 SDA1
-Text GLabel 7750 1550 0    50   Input ~ 0
+Text GLabel 8550 1550 0    50   Input ~ 0
 SCL1
 Wire Wire Line
-	7750 1550 7800 1550
-Wire Wire Line
-	7800 1250 7750 1250
+	8550 1550 8600 1550
+Wire Wire Line
+	8600 1250 8550 1250
 $Comp
 L power:+3.3V #PWR016
 U 1 1 62142CB7
-P 8150 1150
-F 0 "#PWR016" H 8150 1000 50  0001 C CNN
-F 1 "+3.3V" H 8165 1323 50  0000 C CNN
-F 2 "" H 8150 1150 50  0001 C CNN
-F 3 "" H 8150 1150 50  0001 C CNN
-	1    8150 1150
-	1    0    0    -1
-$EndComp
-Wire Wire Line
-	8150 1150 8150 1250
-Wire Wire Line
-	8150 1250 8100 1250
-Wire Wire Line
-	8100 1550 8150 1550
-Wire Wire Line
-	8150 1550 8150 1250
-Connection ~ 8150 1250
+P 8950 1150
+F 0 "#PWR016" H 8950 1000 50  0001 C CNN
+F 1 "+3.3V" H 8965 1323 50  0000 C CNN
+F 2 "" H 8950 1150 50  0001 C CNN
+F 3 "" H 8950 1150 50  0001 C CNN
+	1    8950 1150
+	1    0    0    -1
+$EndComp
+Wire Wire Line
+	8950 1150 8950 1250
+Wire Wire Line
+	8950 1250 8900 1250
+Wire Wire Line
+	8900 1550 8950 1550
+Wire Wire Line
+	8950 1550 8950 1250
+Connection ~ 8950 1250
 $Comp
 L Device:R R11
 U 1 1 6213D612
-P 7950 1550
-F 0 "R11" V 7743 1550 50  0000 C CNN
-F 1 "4k7" V 7834 1550 50  0000 C CNN
-F 2 "Resistor_SMD:R_0805_2012Metric_Pad1.20x1.40mm_HandSolder" V 7880 1550 50  0001 C CNN
-F 3 "~" H 7950 1550 50  0001 C CNN
-	1    7950 1550
+P 8750 1550
+F 0 "R11" V 8543 1550 50  0000 C CNN
+F 1 "4k7" V 8634 1550 50  0000 C CNN
+F 2 "Resistor_SMD:R_0805_2012Metric_Pad1.20x1.40mm_HandSolder" V 8680 1550 50  0001 C CNN
+F 3 "~" H 8750 1550 50  0001 C CNN
+	1    8750 1550
 	0    1    1    0
 $EndComp
@@
 L Device:R R10
 U 1 1 6213CF4B
-P 7950 1250
-F 0 "R10" V 7743 1250 50  0000 C CNN
-F 1 "4k7" V 7834 1250 50  0000 C CNN
-F 2 "Resistor_SMD:R_0805_2012Metric_Pad1.20x1.40mm_HandSolder" V 7880 1250 50  0001 C CNN
-F 3 "~" H 7950 1250 50  0001 C CNN
-	1    7950 1250
+P 8750 1250
+F 0 "R10" V 8543 1250 50  0000 C CNN
+F 1 "4k7" V 8634 1250 50  0000 C CNN
+F 2 "Resistor_SMD:R_0805_2012Metric_Pad1.20x1.40mm_HandSolder" V 8680 1250 50  0001 C CNN
+F 3 "~" H 8750 1250 50  0001 C CNN
+	1    8750 1250
 	0    1    1    0
 $EndComp
@@
 Arduino Header connectors
 Wire Notes Line
-	7250 750  8450 750
-Text Notes 7250 700  0    50   ~ 0
+	8050 750  9250 750
+Text Notes 8050 700  0    50   ~ 0
 data
 Text Notes 700  4400 0    50   ~ 0
@@
 F1 "STM32L151RET6TR.sch" 50
 $EndSheet
-Text GLabel 7750 2150 0    50   Input ~ 0
+Text GLabel 8550 2150 0    50   Input ~ 0
 SDA2
-Text GLabel 7750 2450 0    50   Input ~ 0
+Text GLabel 8550 2450 0    50   Input ~ 0
 SCL2
 Wire Wire Line
-	7750 2450 7800 2450
-Wire Wire Line
-	7800 2150 7750 2150
+	8550 2450 8600 2450
+Wire Wire Line
+	8600 2150 8550 2150
 $Comp
 L power:+3.3V #PWR0103
 U 1 1 62898F4E
-P 8150 2050
-F 0 "#PWR0103" H 8150 1900 50  0001 C CNN
-F 1 "+3.3V" H 8165 2223 50  0000 C CNN
-F 2 "" H 8150 2050 50  0001 C CNN
-F 3 "" H 8150 2050 50  0001 C CNN
-	1    8150 2050
-	1    0    0    -1
-$EndComp
-Wire Wire Line
-	8150 2050 8150 2150
-Wire Wire Line
-	8150 2150 8100 2150
-Wire Wire Line
-	8100 2450 8150 2450
-Wire Wire Line
-	8150 2450 8150 2150
-Connection ~ 8150 2150
+P 8950 2050
+F 0 "#PWR0103" H 8950 1900 50  0001 C CNN
+F 1 "+3.3V" H 8965 2223 50  0000 C CNN
+F 2 "" H 8950 2050 50  0001 C CNN
+F 3 "" H 8950 2050 50  0001 C CNN
+	1    8950 2050
+	1    0    0    -1
+$EndComp
+Wire Wire Line
+	8950 2050 8950 2150
+Wire Wire Line
+	8950 2150 8900 2150
+Wire Wire Line
+	8900 2450 8950 2450
+Wire Wire Line
+	8950 2450 8950 2150
+Connection ~ 8950 2150
 $Comp
 L Device:R R22
 U 1 1 62898F59
-P 7950 2450
-F 0 "R22" V 7743 2450 50  0000 C CNN
-F 1 "4k7" V 7834 2450 50  0000 C CNN
-F 2 "Resistor_SMD:R_0805_2012Metric_Pad1.20x1.40mm_HandSolder" V 7880 2450 50  0001 C CNN
-F 3 "~" H 7950 2450 50  0001 C CNN
-	1    7950 2450
+P 8750 2450
+F 0 "R22" V 8543 2450 50  0000 C CNN
+F 1 "4k7" V 8634 2450 50  0000 C CNN
+F 2 "Resistor_SMD:R_0805_2012Metric_Pad1.20x1.40mm_HandSolder" V 8680 2450 50  0001 C CNN
+F 3 "~" H 8750 2450 50  0001 C CNN
+	1    8750 2450
 	0    1    1    0
 $EndComp
@@
 L Device:R R21
 U 1 1 62898F5F
-P 7950 2150
-F 0 "R21" V 7743 2150 50  0000 C CNN
-F 1 "4k7" V 7834 2150 50  0000 C CNN
-F 2 "Resistor_SMD:R_0805_2012Metric_Pad1.20x1.40mm_HandSolder" V 7880 2150 50  0001 C CNN
-F 3 "~" H 7950 2150 50  0001 C CNN
-	1    7950 2150
-	0    1    1    0
-$EndComp
-Wire Notes Line
-	8450 2800 7250 2800
-Wire Notes Line
-	8450 750  8450 2800
-Wire Notes Line
-	7250 750  7250 2800
+P 8750 2150
+F 0 "R21" V 8543 2150 50  0000 C CNN
+F 1 "4k7" V 8634 2150 50  0000 C CNN
+F 2 "Resistor_SMD:R_0805_2012Metric_Pad1.20x1.40mm_HandSolder" V 8680 2150 50  0001 C CNN
+F 3 "~" H 8750 2150 50  0001 C CNN
+	1    8750 2150
+	0    1    1    0
+$EndComp
+Wire Notes Line
+	9250 2800 8050 2800
+Wire Notes Line
+	9250 750  9250 2800
+Wire Notes Line
+	8050 750  8050 2800
 Wire Notes Line
 	2000 5850 2000 6850
@@
 L power:+3.3V #PWR0120
 U 1 1 62250C10
-P 6800 1450
-F 0 "#PWR0120" H 6800 1300 50  0001 C CNN
-F 1 "+3.3V" V 6815 1578 50  0000 L CNN
-F 2 "" H 6800 1450 50  0001 C CNN
-F 3 "" H 6800 1450 50  0001 C CNN
-	1    6800 1450
-	0    1    1    0
+P 6700 1400
+F 0 "#PWR0120" H 6700 1250 50  0001 C CNN
+F 1 "+3.3V" H 6600 1550 50  0000 L CNN
+F 2 "" H 6700 1400 50  0001 C CNN
+F 3 "" H 6700 1400 50  0001 C CNN
+	1    6700 1400
+	1    0    0    -1
 $EndComp
 $Comp
@@
 Wire Wire Line
 	6450 1450 6500 1450
-Wire Wire Line
-	6800 1450 6700 1450
 Connection ~ 6700 1450
 Connection ~ 6500 1450
@@
 $EndComp
 Wire Notes Line
-	3550 4200 7200 4200
-Wire Notes Line
-	7200 4200 7200 750
-Wire Notes Line
 	3550 750  3550 4200
-Wire Notes Line
-	3550 750  7200 750
 Wire Wire Line
 	9600 4200 9750 4200
@@
 Wire Notes Line
 	7250 3600 7250 6500
+$Comp
+L Device:C C11
+U 1 1 62216B61
+P 7100 1650
+F 0 "C11" H 7215 1696 50  0000 L CNN
+F 1 "4.7µF" H 7215 1605 50  0000 L CNN
+F 2 "Capacitor_SMD:C_0805_2012Metric_Pad1.18x1.45mm_HandSolder" H 7138 1500 50  0001 C CNN
+F 3 "~" H 7100 1650 50  0001 C CNN
+	1    7100 1650
+	1    0    0    -1
+$EndComp
+$Comp
+L Device:C C12
+U 1 1 6222AC8B
+P 7550 1650
+F 0 "C12" H 7665 1696 50  0000 L CNN
+F 1 "4.7µF" H 7665 1605 50  0000 L CNN
+F 2 "Capacitor_SMD:C_0805_2012Metric_Pad1.18x1.45mm_HandSolder" H 7588 1500 50  0001 C CNN
+F 3 "~" H 7550 1650 50  0001 C CNN
+	1    7550 1650
+	1    0    0    -1
+$EndComp
+Wire Wire Line
+	6700 1400 6700 1450
+Wire Wire Line
+	7100 1450 7100 1500
+Wire Wire Line
+	6700 1450 7100 1450
+Wire Wire Line
+	7100 1450 7550 1450
+Wire Wire Line
+	7550 1450 7550 1500
+Connection ~ 7100 1450
+$Comp
+L power:GND #PWR0198
+U 1 1 62262C04
+P 7100 1800
+F 0 "#PWR0198" H 7100 1550 50  0001 C CNN
+F 1 "GND" H 7105 1627 50  0000 C CNN
+F 2 "" H 7100 1800 50  0001 C CNN
+F 3 "" H 7100 1800 50  0001 C CNN
+	1    7100 1800
+	1    0    0    -1
+$EndComp
+$Comp
+L power:GND #PWR0199
+U 1 1 62263181
+P 7550 1800
+F 0 "#PWR0199" H 7550 1550 50  0001 C CNN
+F 1 "GND" H 7555 1627 50  0000 C CNN
+F 2 "" H 7550 1800 50  0001 C CNN
+F 3 "" H 7550 1800 50  0001 C CNN
+	1    7550 1800
+	1    0    0    -1
+$EndComp
+Wire Notes Line
+	3550 750  7900 750
+Wire Notes Line
+	7900 2250 7150 2250
+Wire Notes Line
+	7150 2250 7150 4200
+Wire Notes Line
+	7900 750  7900 2250
+Wire Notes Line
+	7150 4200 3550 4200
 $EndSCHEMATC

Commit message: add PCB V12
Parts:
- removed JP10, JP11, JP12, JP14, JP5, JP6, JP7, JP8, JP9: SolderJumper_2_Open, Jumper:SolderJumper-2_P1.3mm_Open_Pad1.0x1.5mm, symbol Jumper:SolderJumper_2_Open
- added H10, H11, H12, H13, H14, H15, H16, H7, H8, H9: MountingHole, MountingHole:MountingHole_3.2mm_M3, symbol Mechanical:MountingHole
Connections:
- net _XSHUT_0 is gone; now on net XSHUT_3: J4.4 (Pin_4)
- net _XSHUT_2 is gone; now on net GPIOI_2: J5.5 (Pin_5)
- net _XSHUT_3 is gone; now on net SW_1: J4.5 (Pin_5)
- net _XSHUT_5 is gone; now on net GPIOI_1: J5.4 (Pin_4)
- net _XSHUT_6 is gone; now on net SW_2: J4.6 (Pin_6)
- net _XSHUT_7 is gone; now on net LED_3: J6.5 (Pin_5)
- net _XSHUT_8 is gone; now on net GPIOI_0: J5.3 (Pin_3)
- net GPIOI_0: no longer J4.1 (Pin_1)
- net GPIOI_1: no longer J4.2 (Pin_2)
- net GPIOI_2: no longer J4.3 (Pin_3)
- net LED_1: now also J6.7 (Pin_7); no longer J5.2 (Pin_2)
- net LED_2: now also J6.6 (Pin_6); no longer J6.7 (Pin_7)
- net LED_3: no longer J6.6 (Pin_6)
- net XSHUT_0: now also J4.1 (Pin_1)
- net XSHUT_1: now also J4.2 (Pin_2)
- net XSHUT_2: now also J4.3 (Pin_3)
- net GPIOI_3: now reaches J5.6 (Pin_6)
- net _XSHUT_1: no longer names the net of J5.1 (Pin_1)
- net _XSHUT_4: no longer names the net of J6.8 (Pin_8)
Other:
- moved on the sheet: H1, H2, H3, H4, H5, H6

Commit message: cleanup PCB V0.1
Other:
- moved on the sheet: J3, J4, J5, J6, R10, R11, R21, R22
