File: pcb/GestureControl/STM32F401RET6U.sch (KiCad schematic (older format))
At the start: 22 parts, among them J7 Conn_01x09, SW3 SW_Push_Dual, U6 STM32F401RETx, Y1 8MHz, Y2 32kHz

Commit message: add
Parts:
- removed J7: Conn_01x09, Connector_PinHeader_2.54mm:PinHeader_1x09_P2.54mm_Vertical, symbol Connector_Generic:Conn_01x09
- removed U6: STM32F401RETx, Package_QFP:LQFP-64_10x10mm_P0.5mm, symbol MCU_ST_STM32F4:STM32F401RETx
- added C31: 100n, Capacitor_SMD:C_0603_1608Metric_Pad1.08x0.95mm_HandSolder, symbol Device:C
- added C32: 1µ, Capacitor_SMD:C_0805_2012Metric_Pad1.18x1.45mm_HandSolder, symbol Device:C
- added J7: FTDI, Connector_PinHeader_2.54mm:PinHeader_1x06_P2.54mm_Vertical, symbol Connector_Generic:Conn_01x06
- added J8: Serial Wire, Connector_PinHeader_2.54mm:PinHeader_1x05_P2.54mm_Vertical, symbol Connector_Generic:Conn_01x05
- added J9: USB, symbol Connector_Generic:Conn_01x04
- added SW4: BOOT, Button_Switch_SMD:SW_Push_1P1T_NO_6x6mm_H9.5mm, symbol Switch:SW_Push_Dual
- added TP?: SDA_TEST, symbol Connector:TestPoint
- added TP?: SCL_TEST, symbol Connector:TestPoint
- added U6: STM32L151RETx, Package_QFP:LQFP-64_10x10mm_P0.5mm, symbol MCU_ST_STM32L1:STM32L151RETx
- added U?: STM32L151ZCTx, Package_QFP:LQFP-144_20x20mm_P0.5mm, symbol MCU_ST_STM32L1:STM32L151ZCTx
- added U?: STM32F723ZETx, Package_QFP:LQFP-144_20x20mm_P0.5mm, symbol MCU_ST_STM32F7:STM32F723ZETx
- C15, C22, C25, C26, C27, C28, C29: footprint Capacitor_SMD:C_0805_2012Metric_Pad1.18x1.45mm_HandSolder -> Capacitor_SMD:C_0603_1608Metric_Pad1.08x0.95mm_HandSolder
- C18: value 4.3p -> 20p; footprint Capacitor_SMD:C_0805_2012Metric_Pad1.18x1.45mm_HandSolder -> Capacitor_SMD:C_0603_1608Metric_Pad1.08x0.95mm_HandSolder
- C19: value 4,3p -> 20p; footprint Capacitor_SMD:C_0805_2012Metric_Pad1.18x1.45mm_HandSolder -> Capacitor_SMD:C_0603_1608Metric_Pad1.08x0.95mm_HandSolder
- C20, C21: value 2,2µ -> 100n; footprint Capacitor_SMD:C_0805_2012Metric_Pad1.18x1.45mm_HandSolder -> Capacitor_SMD:C_0603_1608Metric_Pad1.08x0.95mm_HandSolder
- C30: footprint (none) -> Capacitor_SMD:C_0805_2012Metric_Pad1.18x1.45mm_HandSolder
- SW3: value SW_Push_Dual -> RST; footprint (none) -> Button_Switch_SMD:SW_Push_1P1T_NO_6x6mm_H9.5mm
- Y1: footprint (none) -> Crystal:Crystal_SMD_HC49-SD
- Y2: footprint (none) -> Crystal:Crystal_SMD_SeikoEpson_MC306-4Pin_8.0x3.2mm
Connections:
- net labels added: +5V, BOOT, FTDI_CTS, FTDI_RTS, FTDI_RXD, FTDI_TXD, OS32_IN, OS32_OUT, SWCLK, SWDAT, USB_DN, USB_DP
- net labels removed: OS_IN, OS_OUT, TCK, TMS, USART_RX, USART_TX
- wire segments 137 -> 118
- no-connect marks 29 -> 0

Commit message: new PCB
Parts:
- J7: footprint Connector_PinHeader_2.54mm:PinHeader_1x06_P2.54mm_Vertical -> Connector_PinHeader_2.54mm:PinHeader_1x06_P2.54mm_Horizontal
- J8: footprint Connector_PinHeader_2.54mm:PinHeader_1x05_P2.54mm_Vertical -> Connector_PinHeader_2.54mm:PinHeader_1x05_P2.54mm_Horizontal
- TP1, TP2: renamed from TP?; footprint (none) -> TestPoint:TestPoint_Pad_1.0x1.0mm
- gave numbers to parts that had none: 2
- renumbered C16 to C17, C17 to C18, C18 to C19, C15 to C21, C19 to C22, C21 to C23, C22 to C24, C31 to C28, C28 to C29, C32 to C30, C29 to C31, C30 to C32, R16 to R18, R17 to R19, R18 to R20, SW4 to SW3, SW3 to SW4
