File: pcb/GestureControl/VL53L3CX_RIGHT.sch (KiCad schematic (older format))
At the start: 6 parts, among them U4 VL53L3CXV0DH_RIGHT

Commit message: add
Parts:
- C10, C9: footprint Capacitor_SMD:C_0805_2012Metric_Pad1.18x1.45mm_HandSolder -> Capacitor_SMD:C_0603_1608Metric_Pad1.08x0.95mm_HandSolder
Changed lines of the file:
@@
 F 0 "C10" H 6665 3896 50  0000 L CNN
 F 1 "100n" H 6665 3805 50  0000 L CNN
-F 2 "Capacitor_SMD:C_0805_2012Metric_Pad1.18x1.45mm_HandSolder" H 6588 3700 50  0001 C CNN
+F 2 "Capacitor_SMD:C_0603_1608Metric_Pad1.08x0.95mm_HandSolder" H 6588 3700 50  0001 C CNN
 F 3 "~" H 6550 3850 50  0001 C CNN
 	1    6550 3850
@@
 F 0 "C9" H 3215 3896 50  0000 L CNN
 F 1 "100n" H 3215 3805 50  0000 L CNN
-F 2 "Capacitor_SMD:C_0805_2012Metric_Pad1.18x1.45mm_HandSolder" H 3138 3700 50  0001 C CNN
+F 2 "Capacitor_SMD:C_0603_1608Metric_Pad1.08x0.95mm_HandSolder" H 3138 3700 50  0001 C CNN
 F 3 "~" H 3100 3850 50  0001 C CNN
 	1    3100 3850

Commit message: new PCB
Parts:
- U4: footprint VL53L3CX:VL53L3CXV0DH&slash_1 -> VL53L3C1:VL53L3CXV0DH&slash_1
- renumbered C9 to C11, C10 to C12, C11 to C13, R12 to R14, R13 to R15
Connections:
- net SCL renamed SCL1
- net SDA renamed SDA1
Changed lines of the file:
@@
 F 0 "U4" H 4850 4087 60  0000 C CNN
 F 1 "VL53L3CXV0DH_RIGHT" H 4850 3981 60  0000 C CNN
-F 2 "VL53L3CX:VL53L3CXV0DH&slash_1" H 4850 3940 60  0001 C CNN
+F 2 "VL53L3C1:VL53L3CXV0DH&slash_1" H 4850 3940 60  0001 C CNN
 F 3 "" H 3850 3700 60  0000 C CNN
 	1    3850 3700
@@
 P 5900 3800
 AR Path="/62398514/623B5A74" Ref="#PWR?"  Part="1"
-AR Path="/623A41A0/623B5A74" Ref="#PWR0132"  Part="1"
-F 0 "#PWR0132" H 5900 3650 50  0001 C CNN
+AR Path="/623A41A0/623B5A74" Ref="#PWR044"  Part="1"
+F 0 "#PWR044" H 5900 3650 50  0001 C CNN
 F 1 "+3.3V" V 5915 3928 50  0000 L CNN
 F 2 "" H 5900 3800 50  0001 C CNN
@@
 P 5900 3700
 AR Path="/62398514/623B5A7A" Ref="#PWR?"  Part="1"
-AR Path="/623A41A0/623B5A7A" Ref="#PWR0133"  Part="1"
-F 0 "#PWR0133" H 5900 3450 50  0001 C CNN
+AR Path="/623A41A0/623B5A7A" Ref="#PWR043"  Part="1"
+F 0 "#PWR043" H 5900 3450 50  0001 C CNN
 F 1 "GND" V 5905 3572 50  0000 R CNN
 F 2 "" H 5900 3700 50  0001 C CNN
@@
 $EndComp
 Text GLabel 5900 3900 2    50   Input ~ 0
-SCL
+SCL1
 Text GLabel 5900 4000 2    50   Input ~ 0
-SDA
+SDA1
 $Comp
 L power:+3.3V #PWR?
@@
 P 3800 3700
 AR Path="/62398514/623B5A82" Ref="#PWR?"  Part="1"
-AR Path="/623A41A0/623B5A82" Ref="#PWR0134"  Part="1"
-F 0 "#PWR0134" H 3800 3550 50  0001 C CNN
+AR Path="/623A41A0/623B5A82" Ref="#PWR038"  Part="1"
+F 0 "#PWR038" H 3800 3550 50  0001 C CNN
 F 1 "+3.3V" V 3815 3828 50  0000 L CNN
 F 2 "" H 3800 3700 50  0001 C CNN
@@
 P 3800 3900
 AR Path="/62398514/623B5A88" Ref="#PWR?"  Part="1"
-AR Path="/623A41A0/623B5A88" Ref="#PWR0135"  Part="1"
-F 0 "#PWR0135" H 3800 3650 50  0001 C CNN
+AR Path="/623A41A0/623B5A88" Ref="#PWR040"  Part="1"
+F 0 "#PWR040" H 3800 3650 50  0001 C CNN
 F 1 "GND" V 3805 3772 50  0000 R CNN
 F 2 "" H 3800 3900 50  0001 C CNN
@@
 P 3800 4000
 AR Path="/62398514/623B5A8E" Ref="#PWR?"  Part="1"
-AR Path="/623A41A0/623B5A8E" Ref="#PWR0136"  Part="1"
-F 0 "#PWR0136" H 3800 3750 50  0001 C CNN
+AR Path="/623A41A0/623B5A8E" Ref="#PWR041"  Part="1"
+F 0 "#PWR041" H 3800 3750 50  0001 C CNN
 F 1 "GND" V 3805 3872 50  0000 R CNN
 F 2 "" H 3800 4000 50  0001 C CNN
@@
 P 3800 4200
 AR Path="/62398514/623B5A94" Ref="#PWR?"  Part="1"
-AR Path="/623A41A0/623B5A94" Ref="#PWR0137"  Part="1"
-F 0 "#PWR0137" H 3800 3950 50  0001 C CNN
+AR Path="/623A41A0/623B5A94" Ref="#PWR042"  Part="1"
+F 0 "#PWR042" H 3800 3950 50  0001 C CNN
 F 1 "GND" V 3805 4072 50  0000 R CNN
 F 2 "" H 3800 4200 50  0001 C CNN
@@
 P 3800 3800
 AR Path="/62398514/623B5A9B" Ref="#PWR?"  Part="1"
-AR Path="/623A41A0/623B5A9B" Ref="#PWR0138"  Part="1"
-F 0 "#PWR0138" H 3800 3550 50  0001 C CNN
+AR Path="/623A41A0/623B5A9B" Ref="#PWR039"  Part="1"
+F 0 "#PWR039" H 3800 3550 50  0001 C CNN
 F 1 "GND" V 3805 3672 50  0000 R CNN
 F 2 "" H 3800 3800 50  0001 C CNN
@@
 P 6550 3850
 AR Path="/62398514/623B5AAC" Ref="C?"  Part="1"
-AR Path="/623A41A0/623B5AAC" Ref="C10"  Part="1"
-F 0 "C10" H 6665 3896 50  0000 L CNN
+AR Path="/623A41A0/623B5AAC" Ref="C12"  Part="1"
+F 0 "C12" H 6665 3896 50  0000 L CNN
 F 1 "100n" H 6665 3805 50  0000 L CNN
 F 2 "Capacitor_SMD:C_0603_1608Metric_Pad1.08x0.95mm_HandSolder" H 6588 3700 50  0001 C CNN
@@
 P 7000 3850
 AR Path="/62398514/623B5AB2" Ref="C?"  Part="1"
-AR Path="/623A41A0/623B5AB2" Ref="C11"  Part="1"
-F 0 "C11" H 7115 3896 50  0000 L CNN
+AR Path="/623A41A0/623B5AB2" Ref="C13"  Part="1"
+F 0 "C13" H 7115 3896 50  0000 L CNN
 F 1 "4.7µ" H 7115 3805 50  0000 L CNN
 F 2 "Capacitor_SMD:C_0805_2012Metric_Pad1.18x1.45mm_HandSolder" H 7038 3700 50  0001 C CNN
@@
 P 6550 3650
 AR Path="/62398514/623B5AB8" Ref="#PWR?"  Part="1"
-AR Path="/623A41A0/623B5AB8" Ref="#PWR0139"  Part="1"
-F 0 "#PWR0139" H 6550 3500 50  0001 C CNN
+AR Path="/623A41A0/623B5AB8" Ref="#PWR045"  Part="1"
+F 0 "#PWR045" H 6550 3500 50  0001 C CNN
 F 1 "+3.3V" H 6565 3823 50  0000 C CNN
 F 2 "" H 6550 3650 50  0001 C CNN
@@
 P 7000 3650
 AR Path="/62398514/623B5ABE" Ref="#PWR?"  Part="1"
-AR Path="/623A41A0/623B5ABE" Ref="#PWR0140"  Part="1"
-F 0 "#PWR0140" H 7000 3500 50  0001 C CNN
+AR Path="/623A41A0/623B5ABE" Ref="#PWR047"  Part="1"
+F 0 "#PWR047" H 7000 3500 50  0001 C CNN
 F 1 "+3.3V" H 7015 3823 50  0000 C CNN
 F 2 "" H 7000 3650 50  0001 C CNN
@@
 P 6550 4050
 AR Path="/62398514/623B5AC4" Ref="#PWR?"  Part="1"
-AR Path="/623A41A0/623B5AC4" Ref="#PWR0141"  Part="1"
-F 0 "#PWR0141" H 6550 3800 50  0001 C CNN
+AR Path="/623A41A0/623B5AC4" Ref="#PWR046"  Part="1"
+F 0 "#PWR046" H 6550 3800 50  0001 C CNN
 F 1 "GND" H 6555 3877 50  0000 C CNN
 F 2 "" H 6550 4050 50  0001 C CNN
@@
 P 7000 4050
 AR Path="/62398514/623B5ACA" Ref="#PWR?"  Part="1"
-AR Path="/623A41A0/623B5ACA" Ref="#PWR0142"  Part="1"
-F 0 "#PWR0142" H 7000 3800 50  0001 C CNN
+AR Path="/623A41A0/623B5ACA" Ref="#PWR048"  Part="1"
+F 0 "#PWR048" H 7000 3800 50  0001 C CNN
 F 1 "GND" H 7005 3877 50  0000 C CNN
 F 2 "" H 7000 4050 50  0001 C CNN
@@
 P 8000 3900
 AR Path="/62398514/623B5AD0" Ref="R?"  Part="1"
-AR Path="/623A41A0/623B5AD0" Ref="R13"  Part="1"
-F 0 "R13" V 7793 3900 50  0000 C CNN
+AR Path="/623A41A0/623B5AD0" Ref="R15"  Part="1"
+F 0 "R15" V 7793 3900 50  0000 C CNN
 F 1 "10k" V 7884 3900 50  0000 C CNN
 F 2 "Resistor_SMD:R_0805_2012Metric_Pad1.20x1.40mm_HandSolder" V 7930 3900 50  0001 C CNN
@@
 P 8000 3600
 AR Path="/62398514/623B5AD6" Ref="R?"  Part="1"
-AR Path="/623A41A0/623B5AD6" Ref="R12"  Part="1"
-F 0 "R12" V 7793 3600 50  0000 C CNN
+AR Path="/623A41A0/623B5AD6" Ref="R14"  Part="1"
+F 0 "R14" V 7793 3600 50  0000 C CNN
 F 1 "10k" V 7884 3600 50  0000 C CNN
 F 2 "Resistor_SMD:R_0805_2012Metric_Pad1.20x1.40mm_HandSolder" V 7930 3600 50  0001 C CNN
@@
 P 8200 3600
 AR Path="/62398514/623B5ADE" Ref="#PWR?"  Part="1"
-AR Path="/623A41A0/623B5ADE" Ref="#PWR0143"  Part="1"
-F 0 "#PWR0143" H 8200 3450 50  0001 C CNN
+AR Path="/623A41A0/623B5ADE" Ref="#PWR049"  Part="1"
+F 0 "#PWR049" H 8200 3450 50  0001 C CNN
 F 1 "+3.3V" V 8215 3728 50  0000 L CNN
 F 2 "" H 8200 3600 50  0001 C CNN
@@
 P 8200 3900
 AR Path="/62398514/623B5AE4" Ref="#PWR?"  Part="1"
-AR Path="/623A41A0/623B5AE4" Ref="#PWR0144"  Part="1"
-F 0 "#PWR0144" H 8200 3750 50  0001 C CNN
+AR Path="/623A41A0/623B5AE4" Ref="#PWR050"  Part="1"
+F 0 "#PWR050" H 8200 3750 50  0001 C CNN
 F 1 "+3.3V" V 8215 4028 50  0000 L CNN
 F 2 "" H 8200 3900 50  0001 C CNN
@@
 P 3100 3850
 AR Path="/62398514/623B5AF2" Ref="C?"  Part="1"
-AR Path="/623A41A0/623B5AF2" Ref="C9"  Part="1"
-F 0 "C9" H 3215 3896 50  0000 L CNN
+AR Path="/623A41A0/623B5AF2" Ref="C11"  Part="1"
+F 0 "C11" H 3215 3896 50  0000 L CNN
 F 1 "100n" H 3215 3805 50  0000 L CNN
 F 2 "Capacitor_SMD:C_0603_1608Metric_Pad1.08x0.95mm_HandSolder" H 3138 3700 50  0001 C CNN
@@
 P 3100 3650
 AR Path="/62398514/623B5AF8" Ref="#PWR?"  Part="1"
-AR Path="/623A41A0/623B5AF8" Ref="#PWR0145"  Part="1"
-F 0 "#PWR0145" H 3100 3500 50  0001 C CNN
+AR Path="/623A41A0/623B5AF8" Ref="#PWR036"  Part="1"
+F 0 "#PWR036" H 3100 3500 50  0001 C CNN
 F 1 "+3.3V" H 3115 3823 50  0000 C CNN
 F 2 "" H 3100 3650 50  0001 C CNN
@@
 P 3100 4050
 AR Path="/62398514/623B5AFE" Ref="#PWR?"  Part="1"
-AR Path="/623A41A0/623B5AFE" Ref="#PWR0146"  Part="1"
-F 0 "#PWR0146" H 3100 3800 50  0001 C CNN
+AR Path="/623A41A0/623B5AFE" Ref="#PWR037"  Part="1"
+F 0 "#PWR037" H 3100 3800 50  0001 C CNN
 F 1 "GND" H 3105 3877 50  0000 C CNN
 F 2 "" H 3100 4050 50  0001 C CNN

Commit message: add lib inside PCB
Parts:
- U4: footprint VL53L3C1:VL53L3CXV0DH&slash_1 -> VL53L3CX:VL53L3CXV0DH&slash_1
Changed lines of the file:
@@
 AR Path="/62398514/623B5A6D" Ref="U?"  Part="1"
 AR Path="/623A41A0/623B5A6D" Ref="U4"  Part="1"
+AR Path="/623B5A6D" Ref="U4"  Part="1"
 F 0 "U4" H 4850 4087 60  0000 C CNN
 F 1 "VL53L3CXV0DH_RIGHT" H 4850 3981 60  0000 C CNN
-F 2 "VL53L3C1:VL53L3CXV0DH&slash_1" H 4850 3940 60  0001 C CNN
+F 2 "VL53L3CX:VL53L3CXV0DH&slash_1" H 4850 3940 60  0001 C CNN
 F 3 "" H 3850 3700 60  0000 C CNN
 	1    3850 3700

Commit message: add feedback Philip
Parts:
- added C39, C40, C49, C50: 100n, Capacitor_SMD:C_0603_1608Metric_Pad1.08x0.95mm_HandSolder, symbol Device:C
- added C41, C42: 4.7µ, Capacitor_SMD:C_0805_2012Metric_Pad1.18x1.45mm_HandSolder, symbol Device:C
- added U10, U8: VL53L3CXV0DH_RIGHT, VL53L3CX:VL53L3CXV0DH&slash_1, symbol VL53L3CX:VL53L3CXV0DH_1
Connections:
- net +3V3: now also C39.1, C40.1, C41.1, C42.1, C49.1, C50.1, U10.1 (AVDDVCSEL), U10.11 (AVDD), U8.1 (AVDDVCSEL), U8.11 (AVDD)
- net GND: now also C39.2, C40.2, C41.2, C42.2, C49.2, C50.2, U10.12 (GND4), U10.2 (AVSSVCSEL), U10.3 (GND), U10.4 (GND2), U10.6 (GND3), U8.12 (GND4), U8.2 (AVSSVCSEL), U8.3 (GND), U8.4 (GND2), U8.6 (GND3)
- net GPIOI_2: now also U10.7 (GPIO1), U8.7 (GPIO1)
- net SCL1: now also U10.10 (SCL), U8.10 (SCL)
- net SDA1: now also U10.9 (SDA), U8.9 (SDA)
- net XSHUT_2: now also U10.5 (XSHUT), U8.5 (XSHUT)
- net at U4.8 (DNC): now also U10.8 (DNC), U8.8 (DNC)

Commit message: add PCBV0.11
Parts:
- removed C11, C12: 100n, Capacitor_SMD:C_0603_1608Metric_Pad1.08x0.95mm_HandSolder, symbol Device:C
- removed C13: 4.7µ, Capacitor_SMD:C_0805_2012Metric_Pad1.18x1.45mm_HandSolder, symbol Device:C
- removed R14, R15: 10k, Resistor_SMD:R_0805_2012Metric_Pad1.20x1.40mm_HandSolder, symbol Device:R
- added C53, C54, C55: 4.7µ, Capacitor_SMD:C_0805_2012Metric_Pad1.18x1.45mm_HandSolder, symbol Device:C
- added JP27, JP28, JP29, JP30, JP31, JP32, JP33, JP34, JP35: SolderJumper_2_Open, Jumper:SolderJumper-2_P1.3mm_Open_Pad1.0x1.5mm, symbol Jumper:SolderJumper_2_Open
- added R31, R32, R33, R34: 10k, Resistor_SMD:R_0805_2012Metric_Pad1.20x1.40mm_HandSolder, symbol Device:R
- C41, C42: value 4.7µ -> 100n; footprint Capacitor_SMD:C_0805_2012Metric_Pad1.18x1.45mm_HandSolder -> Capacitor_SMD:C_0603_1608Metric_Pad1.08x0.95mm_HandSolder
Connections:
- net +3V3: now also JP27.1 (A), JP28.1 (A), JP29.1 (A), R31.1; no longer C39.1, C40.1, C41.1, C42.1, C49.1, C50.1, U10.1 (AVDDVCSEL), U10.11 (AVDD), U4.1 (AVDDVCSEL), U4.11 (AVDD), U8.1 (AVDDVCSEL), U8.11 (AVDD)
- net GND: now also C53.2, C54.2, C55.2
- net GPIOI_2: now also R31.2
- net SCL1: now also JP30.2 (B), JP32.2 (B), JP34.2 (B); no longer U10.10 (SCL), U4.10 (SCL), U8.10 (SCL)
- net SDA1: now also JP31.2 (B), JP33.2 (B), JP35.2 (B); no longer U10.9 (SDA), U4.9 (SDA), U8.9 (SDA)
- net XSHUT_2: now also R32.2; no longer U4.5 (XSHUT), U8.5 (XSHUT)
- new net: JP34.1 (A), U8.10 (SCL)
- new net: JP35.1 (A), U8.9 (SDA)
- new net: JP30.1 (A), U10.10 (SCL)
- new net: JP31.1 (A), U10.9 (SDA)
- new net: JP32.1 (A), U4.10 (SCL)
- new net: JP33.1 (A), U4.9 (SDA)
- new net PWR0: C39.1, C42.1, C53.1, JP27.2 (B), R32.1, U10.1 (AVDDVCSEL), U10.11 (AVDD)
- new net PWR1: C40.1, C49.1, C54.1, JP28.2 (B), R33.1, U4.1 (AVDDVCSEL), U4.11 (AVDD)
- new net PWR2: C41.1, C50.1, C55.1, JP29.2 (B), R34.1, U8.1 (AVDDVCSEL), U8.11 (AVDD)
- new net XSHUT_5: R33.2, U4.5 (XSHUT)
- new net XSHUT_8: R34.2, U8.5 (XSHUT)
- now unconnected: U10.8 (DNC), U4.8 (DNC), U8.8 (DNC)
Other:
- moved on the sheet: U10, U4, U8

Commit message: add PCB V12
Parts:
- removed C41, C50: 100n, Capacitor_SMD:C_0603_1608Metric_Pad1.08x0.95mm_HandSolder, symbol Device:C
- removed C55: 4.7µ, Capacitor_SMD:C_0805_2012Metric_Pad1.18x1.45mm_HandSolder, symbol Device:C
- removed JP29, JP34, JP35: SolderJumper_2_Open, Jumper:SolderJumper-2_P1.3mm_Open_Pad1.0x1.5mm, symbol Jumper:SolderJumper_2_Open
- removed R34: 10k, Resistor_SMD:R_0805_2012Metric_Pad1.20x1.40mm_HandSolder, symbol Device:R
- removed U8: VL53L3CXV0DH_RIGHT, VL53L3CX:VL53L3CXV0DH&slash_1, symbol VL53L3CX:VL53L3CXV0DH_1
- added J13: 690367291076, WR-MM Female SMT Connector:WR-MM Female SMT Connector, symbol WR-MM_Female_SMT_Connector:690367291076
- added JP13, JP24: SolderJumper_2_Open, Jumper:SolderJumper-2_P1.3mm_Open_Pad1.0x1.5mm, symbol Jumper:SolderJumper_2_Open
Connections:
- net GND: now also J13.1, J13.10, J13.3, J13.5, J13.7
- net GPIOI_2: now also J13.8
- net PWR1: now also J13.9
- net SCL1: now also JP13.2 (B)
- net SDA1: now also JP24.2 (B)
- net XSHUT_5: now also J13.6
- new net: J13.4, JP24.1 (A)
- new net: J13.2, JP13.1 (A)
