File: pcb/GestureControl/VL53L3CX_CENTER.sch (KiCad schematic (older format))
At the start: 6 parts, among them U3 VL53L3CXV0DH_CENTER

Commit message: add
Parts:
- C6, C7: footprint Capacitor_SMD:C_0805_2012Metric_Pad1.18x1.45mm_HandSolder -> Capacitor_SMD:C_0603_1608Metric_Pad1.08x0.95mm_HandSolder
Changed lines of the file:
@@
 F 0 "C7" H 7065 3796 50  0000 L CNN
 F 1 "100n" H 7065 3705 50  0000 L CNN
-F 2 "Capacitor_SMD:C_0805_2012Metric_Pad1.18x1.45mm_HandSolder" H 6988 3600 50  0001 C CNN
+F 2 "Capacitor_SMD:C_0603_1608Metric_Pad1.08x0.95mm_HandSolder" H 6988 3600 50  0001 C CNN
 F 3 "~" H 6950 3750 50  0001 C CNN
 	1    6950 3750
@@
 F 0 "C6" H 3615 3796 50  0000 L CNN
 F 1 "100n" H 3615 3705 50  0000 L CNN
-F 2 "Capacitor_SMD:C_0805_2012Metric_Pad1.18x1.45mm_HandSolder" H 3538 3600 50  0001 C CNN
+F 2 "Capacitor_SMD:C_0603_1608Metric_Pad1.08x0.95mm_HandSolder" H 3538 3600 50  0001 C CNN
 F 3 "~" H 3500 3750 50  0001 C CNN
 	1    3500 3750

Commit message: new PCB
Parts:
- U3: footprint VL53L3CX:VL53L3CXV0DH&slash_1 -> VL53L3C1:VL53L3CXV0DH&slash_1
- renumbered C8 to C10, C6 to C8, C7 to C9, R10 to R12, R11 to R13
Connections:
- net SCL renamed SCL1
- net SDA renamed SDA1
Changed lines of the file:
@@
 F 0 "U3" H 5250 3987 60  0000 C CNN
 F 1 "VL53L3CXV0DH_CENTER" H 5250 3881 60  0000 C CNN
-F 2 "VL53L3CX:VL53L3CXV0DH&slash_1" H 5250 3840 60  0001 C CNN
+F 2 "VL53L3C1:VL53L3CXV0DH&slash_1" H 5250 3840 60  0001 C CNN
 F 3 "" H 4250 3600 60  0000 C CNN
 	1    4250 3600
@@
 GPIOI_1
 $Comp
-L power:+3.3V #PWR0117
+L power:+3.3V #PWR029
 U 1 1 6239ED24
 P 6300 3700
-F 0 "#PWR0117" H 6300 3550 50  0001 C CNN
+F 0 "#PWR029" H 6300 3550 50  0001 C CNN
 F 1 "+3.3V" V 6315 3828 50  0000 L CNN
 F 2 "" H 6300 3700 50  0001 C CNN
@@
 $EndComp
 $Comp
-L power:GND #PWR0118
+L power:GND #PWR028
 U 1 1 6239ED2A
 P 6300 3600
-F 0 "#PWR0118" H 6300 3350 50  0001 C CNN
+F 0 "#PWR028" H 6300 3350 50  0001 C CNN
 F 1 "GND" V 6305 3472 50  0000 R CNN
 F 2 "" H 6300 3600 50  0001 C CNN
@@
 $EndComp
 Text GLabel 6300 3800 2    50   Input ~ 0
-SCL
+SCL1
 Text GLabel 6300 3900 2    50   Input ~ 0
-SDA
-$Comp
-L power:+3.3V #PWR0119
+SDA1
+$Comp
+L power:+3.3V #PWR023
 U 1 1 6239ED32
 P 4200 3600
-F 0 "#PWR0119" H 4200 3450 50  0001 C CNN
+F 0 "#PWR023" H 4200 3450 50  0001 C CNN
 F 1 "+3.3V" V 4215 3728 50  0000 L CNN
 F 2 "" H 4200 3600 50  0001 C CNN
@@
 $EndComp
 $Comp
-L power:GND #PWR0120
+L power:GND #PWR025
 U 1 1 6239ED38
 P 4200 3800
-F 0 "#PWR0120" H 4200 3550 50  0001 C CNN
+F 0 "#PWR025" H 4200 3550 50  0001 C CNN
 F 1 "GND" V 4205 3672 50  0000 R CNN
 F 2 "" H 4200 3800 50  0001 C CNN
@@
 $EndComp
 $Comp
-L power:GND #PWR0121
+L power:GND #PWR026
 U 1 1 6239ED3E
 P 4200 3900
-F 0 "#PWR0121" H 4200 3650 50  0001 C CNN
+F 0 "#PWR026" H 4200 3650 50  0001 C CNN
 F 1 "GND" V 4205 3772 50  0000 R CNN
 F 2 "" H 4200 3900 50  0001 C CNN
@@
 $EndComp
 $Comp
-L power:GND #PWR0122
+L power:GND #PWR027
 U 1 1 6239ED44
 P 4200 4100
-F 0 "#PWR0122" H 4200 3850 50  0001 C CNN
+F 0 "#PWR027" H 4200 3850 50  0001 C CNN
 F 1 "GND" V 4205 3972 50  0000 R CNN
 F 2 "" H 4200 4100 50  0001 C CNN
@@
 XSHUT_1
 $Comp
-L power:GND #PWR0123
+L power:GND #PWR024
 U 1 1 6239ED4B
 P 4200 3700
-F 0 "#PWR0123" H 4200 3450 50  0001 C CNN
+F 0 "#PWR024" H 4200 3450 50  0001 C CNN
 F 1 "GND" V 4205 3572 50  0000 R CNN
 F 2 "" H 4200 3700 50  0001 C CNN
@@
 	4250 4100 4200 4100
 $Comp
-L Device:C C7
+L Device:C C9
 U 1 1 6239ED5C
 P 6950 3750
-F 0 "C7" H 7065 3796 50  0000 L CNN
+F 0 "C9" H 7065 3796 50  0000 L CNN
 F 1 "100n" H 7065 3705 50  0000 L CNN
 F 2 "Capacitor_SMD:C_0603_1608Metric_Pad1.08x0.95mm_HandSolder" H 6988 3600 50  0001 C CNN
@@
 $EndComp
 $Comp
-L Device:C C8
+L Device:C C10
 U 1 1 6239ED62
 P 7400 3750
-F 0 "C8" H 7515 3796 50  0000 L CNN
+F 0 "C10" H 7515 3796 50  0000 L CNN
 F 1 "4.7µ" H 7515 3705 50  0000 L CNN
 F 2 "Capacitor_SMD:C_0805_2012Metric_Pad1.18x1.45mm_HandSolder" H 7438 3600 50  0001 C CNN
@@
 $EndComp
 $Comp
-L power:+3.3V #PWR0124
+L power:+3.3V #PWR030
 U 1 1 6239ED68
 P 6950 3550
-F 0 "#PWR0124" H 6950 3400 50  0001 C CNN
+F 0 "#PWR030" H 6950 3400 50  0001 C CNN
 F 1 "+3.3V" H 6965 3723 50  0000 C CNN
 F 2 "" H 6950 3550 50  0001 C CNN
@@
 $EndComp
 $Comp
-L power:+3.3V #PWR0125
+L power:+3.3V #PWR032
 U 1 1 6239ED6E
 P 7400 3550
-F 0 "#PWR0125" H 7400 3400 50  0001 C CNN
+F 0 "#PWR032" H 7400 3400 50  0001 C CNN
 F 1 "+3.3V" H 7415 3723 50  0000 C CNN
 F 2 "" H 7400 3550 50  0001 C CNN
@@
 $EndComp
 $Comp
-L power:GND #PWR0126
+L power:GND #PWR031
 U 1 1 6239ED74
 P 6950 3950
-F 0 "#PWR0126" H 6950 3700 50  0001 C CNN
+F 0 "#PWR031" H 6950 3700 50  0001 C CNN
 F 1 "GND" H 6955 3777 50  0000 C CNN
 F 2 "" H 6950 3950 50  0001 C CNN
@@
 $EndComp
 $Comp
-L power:GND #PWR0127
+L power:GND #PWR033
 U 1 1 6239ED7A
 P 7400 3950
-F 0 "#PWR0127" H 7400 3700 50  0001 C CNN
+F 0 "#PWR033" H 7400 3700 50  0001 C CNN
 F 1 "GND" H 7405 3777 50  0000 C CNN
 F 2 "" H 7400 3950 50  0001 C CNN
@@
 $EndComp
 $Comp
-L Device:R R11
+L Device:R R13
 U 1 1 6239ED80
 P 8400 3800
-F 0 "R11" V 8193 3800 50  0000 C CNN
+F 0 "R13" V 8193 3800 50  0000 C CNN
 F 1 "10k" V 8284 3800 50  0000 C CNN
 F 2 "Resistor_SMD:R_0805_2012Metric_Pad1.20x1.40mm_HandSolder" V 8330 3800 50  0001 C CNN
@@
 $EndComp
 $Comp
-L Device:R R10
+L Device:R R12
 U 1 1 6239ED86
 P 8400 3500
-F 0 "R10" V 8193 3500 50  0000 C CNN
+F 0 "R12" V 8193 3500 50  0000 C CNN
 F 1 "10k" V 8284 3500 50  0000 C CNN
 F 2 "Resistor_SMD:R_0805_2012Metric_Pad1.20x1.40mm_HandSolder" V 8330 3500 50  0001 C CNN
@@
 XSHUT_1
 $Comp
-L power:+3.3V #PWR0128
+L power:+3.3V #PWR034
 U 1 1 6239ED8E
 P 8600 3500
-F 0 "#PWR0128" H 8600 3350 50  0001 C CNN
+F 0 "#PWR034" H 8600 3350 50  0001 C CNN
 F 1 "+3.3V" V 8615 3628 50  0000 L CNN
 F 2 "" H 8600 3500 50  0001 C CNN
@@
 $EndComp
 $Comp
-L power:+3.3V #PWR0129
+L power:+3.3V #PWR035
 U 1 1 6239ED94
 P 8600 3800
-F 0 "#PWR0129" H 8600 3650 50  0001 C CNN
+F 0 "#PWR035" H 8600 3650 50  0001 C CNN
 F 1 "+3.3V" V 8615 3928 50  0000 L CNN
 F 2 "" H 8600 3800 50  0001 C CNN
@@
 	8600 3800 8550 3800
 $Comp
-L Device:C C6
+L Device:C C8
 U 1 1 6239EDA2
 P 3500 3750
-F 0 "C6" H 3615 3796 50  0000 L CNN
+F 0 "C8" H 3615 3796 50  0000 L CNN
 F 1 "100n" H 3615 3705 50  0000 L CNN
 F 2 "Capacitor_SMD:C_0603_1608Metric_Pad1.08x0.95mm_HandSolder" H 3538 3600 50  0001 C CNN
@@
 $EndComp
 $Comp
-L power:+3.3V #PWR0130
+L power:+3.3V #PWR021
 U 1 1 6239EDA8
 P 3500 3550
-F 0 "#PWR0130" H 3500 3400 50  0001 C CNN
+F 0 "#PWR021" H 3500 3400 50  0001 C CNN
 F 1 "+3.3V" H 3515 3723 50  0000 C CNN
 F 2 "" H 3500 3550 50  0001 C CNN
@@
 $EndComp
 $Comp
-L power:GND #PWR0131
+L power:GND #PWR022
 U 1 1 6239EDAE
 P 3500 3950
-F 0 "#PWR0131" H 3500 3700 50  0001 C CNN
+F 0 "#PWR022" H 3500 3700 50  0001 C CNN
 F 1 "GND" H 3505 3777 50  0000 C CNN
 F 2 "" H 3500 3950 50  0001 C CNN

Commit message: add lib inside PCB
Parts:
- U3: footprint VL53L3C1:VL53L3CXV0DH&slash_1 -> VL53L3CX:VL53L3CXV0DH&slash_1
Changed lines of the file:
@@
 U 1 1 6239ED1D
 P 4250 3600
+AR Path="/6239ED1D" Ref="U3"  Part="1"
+AR Path="/62398514/6239ED1D" Ref="U3"  Part="1"
 F 0 "U3" H 5250 3987 60  0000 C CNN
 F 1 "VL53L3CXV0DH_CENTER" H 5250 3881 60  0000 C CNN
-F 2 "VL53L3C1:VL53L3CXV0DH&slash_1" H 5250 3840 60  0001 C CNN
+F 2 "VL53L3CX:VL53L3CXV0DH&slash_1" H 5250 3840 60  0001 C CNN
 F 3 "" H 4250 3600 60  0000 C CNN
 	1    4250 3600

Commit message: add feedback Philip
Parts:
- added C35, C36, C47, C48: 100n, Capacitor_SMD:C_0603_1608Metric_Pad1.08x0.95mm_HandSolder, symbol Device:C
- added C37, C38: 4.7µ, Capacitor_SMD:C_0805_2012Metric_Pad1.18x1.45mm_HandSolder, symbol Device:C
- added U12, U13: VL53L3CXV0DH_CENTER, VL53L3CX:VL53L3CXV0DH&slash_1, symbol VL53L3CX:VL53L3CXV0DH_1
Connections:
- net +3V3: now also C35.1, C36.1, C37.1, C38.1, C47.1, C48.1, U12.1 (AVDDVCSEL), U12.11 (AVDD), U13.1 (AVDDVCSEL), U13.11 (AVDD)
- net GND: now also C35.2, C36.2, C37.2, C38.2, C47.2, C48.2, U12.12 (GND4), U12.2 (AVSSVCSEL), U12.3 (GND), U12.4 (GND2), U12.6 (GND3), U13.12 (GND4), U13.2 (AVSSVCSEL), U13.3 (GND), U13.4 (GND2), U13.6 (GND3)
- net GPIOI_1: now also U12.7 (GPIO1), U13.7 (GPIO1)
- net SCL1: now also U12.10 (SCL), U13.10 (SCL)
- net SDA1: now also U12.9 (SDA), U13.9 (SDA)
- net XSHUT_1: now also U12.5 (XSHUT), U13.5 (XSHUT)
- net at U3.8 (DNC): now also U12.8 (DNC), U13.8 (DNC)

Commit message: add PCBV0.11
Parts:
- added JP15, JP16, JP17, JP18, JP19, JP20, JP21, JP22, JP23: SolderJumper_2_Open, Jumper:SolderJumper-2_P1.3mm_Open_Pad1.0x1.5mm, symbol Jumper:SolderJumper_2_Open
- added R29, R30: 10k, Resistor_SMD:R_0805_2012Metric_Pad1.20x1.40mm_HandSolder, symbol Device:R
Connections:
- net +3V3: now also JP15.1 (A), JP16.1 (A), JP17.1 (A); no longer C10.1, C35.1, C36.1, C37.1, C38.1, C47.1, C48.1, C8.1, C9.1, R13.1, U12.1 (AVDDVCSEL), U12.11 (AVDD), U13.1 (AVDDVCSEL), U13.11 (AVDD), U3.1 (AVDDVCSEL), U3.11 (AVDD)
- net SCL1: now also JP18.2 (B), JP20.2 (B), JP22.2 (B); no longer U12.10 (SCL), U13.10 (SCL), U3.10 (SCL)
- net SDA1: now also JP19.2 (B), JP21.2 (B), JP23.2 (B); no longer U12.9 (SDA), U13.9 (SDA), U3.9 (SDA)
- net XSHUT_1: no longer U12.5 (XSHUT), U3.5 (XSHUT)
- new net: JP22.1 (A), U12.10 (SCL)
- new net: JP23.1 (A), U12.9 (SDA)
- new net: JP18.1 (A), U13.10 (SCL)
- new net: JP19.1 (A), U13.9 (SDA)
- new net: JP20.1 (A), U3.10 (SCL)
- new net: JP21.1 (A), U3.9 (SDA)
- new net PWR0: C35.1, C37.1, C47.1, JP15.2 (B), R13.1, U13.1 (AVDDVCSEL), U13.11 (AVDD)
- new net PWR1: C10.1, C8.1, C9.1, JP16.2 (B), R29.1, U3.1 (AVDDVCSEL), U3.11 (AVDD)
- new net PWR2: C36.1, C38.1, C48.1, JP17.2 (B), R30.1, U12.1 (AVDDVCSEL), U12.11 (AVDD)
- new net XSHUT_4: R29.2, U3.5 (XSHUT)
- new net XSHUT_7: R30.2, U12.5 (XSHUT)
- now unconnected: U12.8 (DNC), U13.8 (DNC), U3.8 (DNC)
Other:
- moved on the sheet: C10, C35, C36, C37, C38, C9, R12, R13, U12, U13

Commit message: add PCB V12
Parts:
- removed C47, C48: 100n, Capacitor_SMD:C_0603_1608Metric_Pad1.08x0.95mm_HandSolder, symbol Device:C
- removed JP15, JP16, JP17, JP18, JP19, JP20, JP21, JP22, JP23: SolderJumper_2_Open, Jumper:SolderJumper-2_P1.3mm_Open_Pad1.0x1.5mm, symbol Jumper:SolderJumper_2_Open
- removed U12, U13: VL53L3CXV0DH_CENTER, VL53L3CX:VL53L3CXV0DH&slash_1, symbol VL53L3CX:VL53L3CXV0DH_1
- added C14, C15, C16, C20, C21: 100n, Capacitor_SMD:C_0603_1608Metric_Pad1.08x0.95mm_HandSolder, symbol Device:C
- added C39, C40, C41, C42: 10µ, Capacitor_SMD:C_1206_3216Metric_Pad1.33x1.80mm_HandSolder, symbol Device:C
- added J13, J14, J15, J16, J20, J21: 690367291076, WR-MM Female SMT Connector:WR-MM_Female_SMT_Connector, symbol WR-MM_Female_SMT_Connector:690367291076
- added R16, R17, R31, R32: 10k, Resistor_SMD:R_0805_2012Metric_Pad1.20x1.40mm_HandSolder, symbol Device:R
- added TP10, TP11, TP12, TP13, TP14, TP15, TP16, TP17, TP18, TP19, TP20, TP3, TP4, TP5, TP6, TP7, TP8, TP9: TestPoint, TestPoint:TestPoint_Pad_D2.0mm, symbol Connector:TestPoint
- added U4, U5, U8: VL53L3CXV0DH_1, VL53L3CX:VL53L3CXV0DH&slash_1, symbol VL53L3CX:VL53L3CXV0DH_1
- C36: value 100n -> 4.7µ; footprint Capacitor_SMD:C_0603_1608Metric_Pad1.08x0.95mm_HandSolder -> Capacitor_SMD:C_0805_2012Metric_Pad1.18x1.45mm_HandSolder
- U3: value VL53L3CXV0DH_CENTER -> VL53L3CXV0DH_1
Connections:
- net PWR0 is gone; now on net +3V3: C35.1, C37.1, R13.1
- net PWR1 is gone; now on net +3V3: C10.1, C8.1, C9.1, R29.1, U3.1 (AVDDVCSEL), U3.11 (AVDD)
- net PWR2 is gone; now on net +3V3: C36.1, C38.1, R30.1
- net +3V3: now also C14.1, C15.1, C16.1, C20.1, C21.1, C39.1, C40.1, C41.1, C42.1, J13.9, J14.9, J15.9, J16.9, J20.9, J21.9, R16.1, R17.1, R31.1, R32.1, TP14.1, TP20.1, TP8.1, U4.1 (AVDDVCSEL), U4.11 (AVDD), U5.1 (AVDDVCSEL), U5.11 (AVDD), U8.1 (AVDDVCSEL), U8.11 (AVDD)
- net GND: now also C14.2, C15.2, C16.2, C20.2, C21.2, C39.2, C40.2, C41.2, C42.2, J13.1, J13.10, J13.3, J13.5, J13.7, J14.1, J14.10, J14.3, J14.5, J14.7, J15.1, J15.10, J15.3, J15.5, J15.7, J16.1, J16.10, J16.3, J16.5, J16.7, J20.1, J20.10, J20.3, J20.5, J20.7, J21.1, J21.10, J21.3, J21.5, J21.7, TP13.1, TP19.1, TP7.1, U4.12 (GND4), U4.2 (AVSSVCSEL), U4.3 (GND), U4.4 (GND2), U4.6 (GND3), U5.12 (GND4), U5.2 (AVSSVCSEL), U5.3 (GND), U5.4 (GND2), U5.6 (GND3), U8.12 (GND4), U8.2 (AVSSVCSEL), U8.3 (GND), U8.4 (GND2), U8.6 (GND3)
- net GPIOI_1: now also J13.8, J16.8, TP6.1, U4.7 (GPIO1); no longer U3.7 (GPIO1)
- net SCL1: now also U3.10 (SCL), J13.2, J14.2, J15.2, J16.2, J20.2, J21.2, TP15.1, TP3.1, TP9.1, U4.10 (SCL), U5.10 (SCL), U8.10 (SCL)
- net SDA1: now also U3.9 (SDA), J13.4, J14.4, J15.4, J16.4, J20.4, J21.4, TP10.1, TP16.1, TP4.1, U4.9 (SDA), U5.9 (SDA), U8.9 (SDA)
- net XSHUT_1: now also R29.2, J13.6, J16.6, TP5.1, U4.5 (XSHUT); no longer R13.2
- net XSHUT_4 renamed XSHUT_0
- net XSHUT_0: now also R32.2; no longer R29.2
- net XSHUT_7 renamed XSHUT_3
- net XSHUT_3: now also J15.6, J21.6, TP17.1, U8.5 (XSHUT)
- new net GPIOI_0: R31.2, U3.7 (GPIO1)
- new net GPIOI_2: J14.8, J20.8, R13.2, TP12.1, U5.7 (GPIO1)
- new net GPIOI_3: J15.8, J21.8, R17.2, TP18.1, U8.7 (GPIO1)
- new net XSHUT_2: J14.6, J20.6, R16.2, TP11.1, U5.5 (XSHUT)
Other:
- moved on the sheet: C10, C8, C9, R12, R29

Commit message: cleanup PCB V0.1
Other:
- moved on the sheet: C10, C14, C15, C16, C20, C21, C35, C36, C37, C38, C39, C40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
