File: pcb/GestureControl/STM32L151RET6TR.kicad_sch (KiCad schematic)
At the start: 33 parts, among them J10 EXTERN I2C, J11 Conn_01x02, J12 Conn_01x02, J17 Conn_01x01, J18 Conn_01x01, J19 Conn_01x01, J7 FTDI, J8 Conn_01x06, J9 UART, U6 STM32L151RETx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

Commit message: add breakoutboard
Connections:
- net XSHUT_4: now reaches U6.24 (PC4)
- net XSHUT_4: now also U7.24 (PC4)
- net GPIOI_4: now reaches U6.37 (PC6)
- net GPIOI_4: now also U7.37 (PC6)

Commit message: add docs
Connections:
- net LED_5 is gone; now on net LED_4: U6.26 (PB0), U7.26 (PB0)
- net LED_1: now also U6.15 (PA1), U7.15 (PA1); no longer U6.14 (PA0), U7.14 (PA0)
- net LED_2: now also U6.22 (PA6), U7.22 (PA6); no longer U6.15 (PA1), U7.15 (PA1)
- net LED_3: now also U6.23 (PA7), U7.23 (PA7); no longer U6.22 (PA6), U7.22 (PA6)
- net LED_4: no longer U6.23 (PA7), U7.23 (PA7)
- new net LED_0: U6.14 (PA0), U7.14 (PA0)
Changed lines of the file:
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@@
     )
   )
-  (global_label "LED_4" (shape input) (at 250.19 60.96 0) (fields_autoplaced)
-    (effects (font (size 1.27 1.27)) (justify left))
-    (property "Intersheet References" "${INTERSHEET_REFS}" (id 0) (at 0 0 0)
-      (effects (font (size 1.27 1.27)) hide)
-    )
-  )
-  (global_label "LED_1" (shape input) (at 193.04 40.64 0) (fields_autoplaced)
-    (effects (font (size 1.27 1.27)) (justify left))
-    (property "Intersheet References" "${INTERSHEET_REFS}" (id 0) (at 0 0 0)
-      (effects (font (size 1.27 1.27)) hide)
+  (global_label "LED_3" (shape input) (at 250.19 60.96 0) (fields_autoplaced)
+    (effects (font (size 1.27 1.27)) (justify left))
+    (property "Intersheet References" "${INTERSHEET_REFS}" (id 0) (at 258.1385 60.8806 0)
+      (effects (font (size 1.27 1.27)) (justify left) hide)
+    )
+  )
+  (global_label "LED_0" (shape input) (at 193.04 40.64 0) (fields_autoplaced)
+    (effects (font (size 1.27 1.27)) (justify left))
+    (property "Intersheet References" "${INTERSHEET_REFS}" (id 0) (at 200.9885 40.5606 0)
+      (effects (font (size 1.27 1.27)) (justify left) hide)
     )
   )
@@
     )
   )
-  (global_label "LED_2" (shape input) (at 193.04 43.18 0) (fields_autoplaced)
-    (effects (font (size 1.27 1.27)) (justify left))
-    (property "Intersheet References" "${INTERSHEET_REFS}" (id 0) (at 0 0 0)
-      (effects (font (size 1.27 1.27)) hide)
+  (global_label "LED_1" (shape input) (at 193.04 43.18 0) (fields_autoplaced)
+    (effects (font (size 1.27 1.27)) (justify left))
+    (property "Intersheet References" "${INTERSHEET_REFS}" (id 0) (at 200.9885 43.1006 0)
+      (effects (font (size 1.27 1.27)) (justify left) hide)
     )
   )
@@
     )
   )
-  (global_label "LED_2" (shape input) (at 250.19 45.72 0) (fields_autoplaced)
-    (effects (font (size 1.27 1.27)) (justify left))
-    (property "Intersheet References" "${INTERSHEET_REFS}" (id 0) (at 0 0 0)
-      (effects (font (size 1.27 1.27)) hide)
-    )
-  )
-  (global_label "LED_3" (shape input) (at 250.19 58.42 0) (fields_autoplaced)
-    (effects (font (size 1.27 1.27)) (justify left))
-    (property "Intersheet References" "${INTERSHEET_REFS}" (id 0) (at 0 0 0)
-      (effects (font (size 1.27 1.27)) hide)
+  (global_label "LED_1" (shape input) (at 250.19 45.72 0) (fields_autoplaced)
+    (effects (font (size 1.27 1.27)) (justify left))
+    (property "Intersheet References" "${INTERSHEET_REFS}" (id 0) (at 258.1385 45.6406 0)
+      (effects (font (size 1.27 1.27)) (justify left) hide)
+    )
+  )
+  (global_label "LED_2" (shape input) (at 250.19 58.42 0) (fields_autoplaced)
+    (effects (font (size 1.27 1.27)) (justify left))
+    (property "Intersheet References" "${INTERSHEET_REFS}" (id 0) (at 258.1385 58.3406 0)
+      (effects (font (size 1.27 1.27)) (justify left) hide)
     )
   )
@@
     )
   )
-  (global_label "LED_1" (shape input) (at 250.19 43.18 0) (fields_autoplaced)
-    (effects (font (size 1.27 1.27)) (justify left))
-    (property "Intersheet References" "${INTERSHEET_REFS}" (id 0) (at 0 0 0)
-      (effects (font (size 1.27 1.27)) hide)
+  (global_label "LED_0" (shape input) (at 250.19 43.18 0) (fields_autoplaced)
+    (effects (font (size 1.27 1.27)) (justify left))
+    (property "Intersheet References" "${INTERSHEET_REFS}" (id 0) (at 258.1385 43.1006 0)
+      (effects (font (size 1.27 1.27)) (justify left) hide)
     )
   )
@@
     )
   )
-  (global_label "LED_4" (shape input) (at 193.04 58.42 0) (fields_autoplaced)
-    (effects (font (size 1.27 1.27)) (justify left))
-    (property "Intersheet References" "${INTERSHEET_REFS}" (id 0) (at 0 0 0)
-      (effects (font (size 1.27 1.27)) hide)
+  (global_label "LED_3" (shape input) (at 193.04 58.42 0) (fields_autoplaced)
+    (effects (font (size 1.27 1.27)) (justify left))
+    (property "Intersheet References" "${INTERSHEET_REFS}" (id 0) (at 200.9885 58.3406 0)
+      (effects (font (size 1.27 1.27)) (justify left) hide)
     )
   )
@@
     )
   )
-  (global_label "LED_5" (shape input) (at 193.04 83.82 0) (fields_autoplaced)
-    (effects (font (size 1.27 1.27)) (justify left))
-    (property "Intersheet References" "${INTERSHEET_REFS}" (id 0) (at 0 0 0)
-      (effects (font (size 1.27 1.27)) hide)
+  (global_label "LED_4" (shape input) (at 193.04 83.82 0) (fields_autoplaced)
+    (effects (font (size 1.27 1.27)) (justify left))
+    (property "Intersheet References" "${INTERSHEET_REFS}" (id 0) (at 200.9885 83.7406 0)
+      (effects (font (size 1.27 1.27)) (justify left) hide)
     )
   )
@@
     )
   )
-  (global_label "LED_3" (shape input) (at 193.04 55.88 0) (fields_autoplaced)
-    (effects (font (size 1.27 1.27)) (justify left))
-    (property "Intersheet References" "${INTERSHEET_REFS}" (id 0) (at 0 0 0)
-      (effects (font (size 1.27 1.27)) hide)
-    )
-  )
-  (global_label "LED_5" (shape input) (at 250.19 86.36 0) (fields_autoplaced)
-    (effects (font (size 1.27 1.27)) (justify left))
-    (property "Intersheet References" "${INTERSHEET_REFS}" (id 0) (at 0 0 0)
-      (effects (font (size 1.27 1.27)) hide)
-    )
-  )
+  (global_label "LED_2" (shape input) (at 193.04 55.88 0) (fields_autoplaced)
+    (effects (font (size 1.27 1.27)) (justify left))
+    (property "Intersheet References" "${INTERSHEET_REFS}" (id 0) (at 200.9885 55.8006 0)
+      (effects (font (size 1.27 1.27)) (justify left) hide)
+    )
+  )
+  (global_label "LED_4" (shape input) (at 250.19 86.36 0) (fields_autoplaced)
+    (effects (font (size 1.27 1.27)) (justify left))
+    (property "Intersheet References" "${INTERSHEET_REFS}" (id 0) (at 258.1385 86.2806 0)
+      (effects (font (size 1.27 1.27)) (justify left) hide)
+    )
+  )

Commit message: edit PCB + add docs
Parts:
- C17, C18: value 20p -> 27p
- C19, C22: value 20p -> 15p
Connections:
- net FTDI_RXD: now also J7.4 (Pin_4); no longer J7.5 (Pin_5)
- net FTDI_TXD: now also J7.5 (Pin_5); no longer J7.4 (Pin_4)
Changed lines of the file:
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@@
   (title_block
     (title "MCU")
-    (date "2022-03-04")
-    (rev "V0.1")
+    (date "2022-05-06")
+    (rev "V0.4")
     (company "AP Hogeschool & ED&A")
   )
@@
     (effects (font (size 1.27 1.27)) (justify left bottom))
   )
-  (label "FTDI_RXD" (at 26.67 57.15 180)
+  (label "FTDI_RXD" (at 26.67 54.61 180)
     (effects (font (size 1.27 1.27)) (justify right bottom))
   )
@@
     (effects (font (size 1.27 1.27)) (justify right bottom))
   )
-  (label "FTDI_TXD" (at 26.67 54.61 180)
+  (label "FTDI_TXD" (at 26.67 57.15 180)
     (effects (font (size 1.27 1.27)) (justify right bottom))
   )
@@
     (in_bom yes) (on_board yes)
     (property "Reference" "C17" (id 0) (at 27.94 115.5192 90))
-    (property "Value" "20p" (id 1) (at 27.94 117.8306 90))
+    (property "Value" "27p" (id 1) (at 27.94 117.8306 90))
     (property "Footprint" "Capacitor_SMD:C_0805_2012Metric_Pad1.18x1.45mm_HandSolder" (id 2) (at 24.13 122.8852 0)
       (effects (font (size 1.27 1.27)) hide)
@@
     (in_bom yes) (on_board yes)
     (property "Reference" "C18" (id 0) (at 27.94 128.2192 90))
-    (property "Value" "20p" (id 1) (at 27.94 130.5306 90))
+    (property "Value" "27p" (id 1) (at 27.94 130.5306 90))
     (property "Footprint" "Capacitor_SMD:C_0805_2012Metric_Pad1.18x1.45mm_HandSolder" (id 2) (at 24.13 135.5852 0)
       (effects (font (size 1.27 1.27)) hide)
@@
       (effects (font (size 1.27 1.27)) (justify left))
     )
-    (property "Value" "20p" (id 1) (at 54.61 124.46 0)
+    (property "Value" "15p" (id 1) (at 54.61 124.46 0)
       (effects (font (size 1.27 1.27)) (justify left))
     )
@@
       (effects (font (size 1.27 1.27)) (justify left))
     )
-    (property "Value" "20p" (id 1) (at 76.581 124.333 0)
-      (effects (font (size 1.27 1.27)) (justify left))
-    )
+    (property "Value" "15p" (id 1) (at 76.581 124.333 0)
+      (effects (font (size 1.27 1.27)) (justify left))
+    )
